File: DB9_USER_IO/Eagle_Gerbers/io2db9.sch (EAGLE design)
At the start: 22 parts

Commit message: Routed finished. Added gerbers
Connections:
- net 1PDOWN: now also RN1B.2; no longer RN1A.2
- net 1PFIRE1: now also RN1A.2; no longer RN1B.2
- net AE15: now also RN1B.1; no longer RN1A.1
- net AH11: now also RN1A.1; no longer RN1B.1
Other:
- moved on the sheet: RN1A, RN1B
Changed lines of the file:
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@@
 <instance part="RN2" gate="C" x="88.9" y="66.04"/>
 <instance part="RN1" gate="D" x="88.9" y="50.8"/>
-<instance part="RN1" gate="B" x="88.9" y="45.72"/>
+<instance part="RN1" gate="A" x="88.9" y="45.72"/>
 <instance part="RN2" gate="B" x="88.9" y="40.64"/>
-<instance part="RN1" gate="A" x="88.9" y="35.56"/>
+<instance part="RN1" gate="B" x="88.9" y="35.56"/>
 <instance part="RN2" gate="A" x="88.9" y="30.48"/>
 <instance part="D7" gate="G$1" x="73.66" y="38.1" rot="R180"/>
@@
 <junction x="73.66" y="45.72"/>
 <label x="58.42" y="45.72" size="1.778" layer="95"/>
-<pinref part="RN1" gate="B" pin="1"/>
+<pinref part="RN1" gate="A" pin="1"/>
 </segment>
 <segment>
@@
 <net name="1PDOWN" class="0">
 <segment>
-<pinref part="RN1" gate="A" pin="2"/>
+<pinref part="RN1" gate="B" pin="2"/>
 <wire x1="93.98" y1="35.56" x2="99.06" y2="35.56" width="0.1524" layer="91"/>
 <label x="93.98" y="35.56" size="1.778" layer="95"/>
@@
 <net name="1PFIRE1" class="0">
 <segment>
-<pinref part="RN1" gate="B" pin="2"/>
+<pinref part="RN1" gate="A" pin="2"/>
 <wire x1="93.98" y1="45.72" x2="99.06" y2="45.72" width="0.1524" layer="91"/>
 <label x="93.98" y="45.72" size="1.778" layer="95"/>
@@
 <junction x="73.66" y="35.56"/>
 <label x="58.42" y="35.56" size="1.778" layer="95"/>
-<pinref part="RN1" gate="A" pin="1"/>
-</segment>
-<segment>
+<pinref part="RN1" gate="B" pin="1"/>
+</segment>
+<segment>
